File: ac608.sch (KiCad schematic (older format))
At the start: 24 parts, among them J1 Conn_01x03, J2 Conn_01x03, J2 Jack-DC, J3 JTAG, P2 Conn_02x20_Odd_Even, P3 Conn_01x04, P4 Conn_01x02, P5 Conn_01x03, P6 Conn_01x03, P7 Conn_02x20_Odd_Even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

Commit message: first commit
Connections:
- net labels added: A9, B1, B16, B9, C15, C16, C2, C9, D1, D15, D16, D9, E11, E16, F1, F13, F14, F15, F16, F2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
- wire segments 58 -> 150
Other:
- moved on the sheet: J1, J2, J?, P2, P7, P8, R7, R8
