File: ac608.sch (KiCad schematic (older format))
At the start: 24 parts, among them J1 Conn_01x03, J2 Conn_01x03, J2 Jack-DC, J3 JTAG, P2 Conn_02x20_Odd_Even, P3 Conn_01x04, P4 Conn_01x02, P5 Conn_01x03, P6 Conn_01x03, P7 Conn_02x20_Odd_Even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

Commit message: first commit
Parts:
- removed E1, E2: 470uF, symbol Device:CP
- removed J2: Jack-DC, symbol Connector:Jack-DC
- removed U1: LM1085-3.3, symbol Regulator_Linear:LM1085-3.3
Connections:
- wire segments 150 -> 134
Other:
- moved on the sheet: J1, J2, P7, P8, R1, R2, R3, R7, R8, S1, S2, S3

Commit message: first commit
Connections:
- net labels added: A8, B8, E1
- wire segments 134 -> 247
Other:
- moved on the sheet: J1, J2, J?, P2, P3, P4, P5, P6, P7, P8, R1, R2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

Commit message: first commit
Parts:
- removed J1, J2: Conn_01x03, symbol Connector_Generic:Conn_01x03
- removed J?: HDMI_A_1.4, symbol Connector:HDMI_A_1.4
- added E? (x2): 470uF, symbol Device:CP
- added J2: Jack-DC, symbol Connector:Jack-DC
- added U1: LM1085-3.3, symbol Regulator_Linear:LM1085-3.3
Connections:
- net labels added: +2V5, LVDS_RXCLK_N, LVDS_RXCLK_P, LVDS_TX1_N, LVDS_TX1_P, LVDS_TX2_N, LVDS_TX2_P, LVDS_TX3_N, LVDS_TX3_P, LVDS_TX4_N, LVDS_TX4_P, LVDS_TX5_N, LVDS_TX5_P
- net labels removed: vdd2.5
- wire segments 247 -> 278
Other:
- note added: "POWER"
- moved on the sheet: J3, J?, P2, P3, P4, P5, P6, P7, P8, R1, R2, R3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

Commit message: first commit
Parts:
- removed J?: Conn_02x03_Odd_Even, symbol Connector_Generic:Conn_02x03_Odd_Even
- removed P8: CAMERA, symbol Connector_Generic:Conn_02x10_Odd_Even
- removed R7, R8: 10K, symbol Device:R
- gave numbers to parts that had none: 2
Connections:
- wire segments 278 -> 277
- no-connect marks 5 -> 3
Other:
- moved on the sheet: P3, P4, P5, P6

Commit message: peripheries updated
Other:
- note added: "AC608_HDMI_V2"
Changed lines of the file:
@@
 encoding utf-8
 Sheet 1 4
-Title ""
-Date ""
-Rev ""
-Comp ""
-Comment1 ""
+Title "AC608 development kit"
+Date "2020-10-25"
+Rev "v1.0"
+Comp "Pavol Risa"
+Comment1 "https://github.com/risapav/ac608"
 Comment2 ""
 Comment3 ""
@@
 $EndDescr
 $Bitmap
-Pos 9650 1900
+Pos 10200 1650
 Scale 1.000000
 Data
@@
 U 5F94D5EB
 F0 "stamp_hole" 50
-F1 "fpga_stamp_hole.sch" 50
+F1 "stamp_hole.sch" 50
 F2 "T14" B L 1700 1100 50
 F3 "T15" B L 1700 1200 50
@@
 	1    0    0    -1
 $EndComp
+Text Notes 600  7700 0    50   ~ 0
+AC608_HDMI_V2
 Wire Bus Line
 	6800 3400 6800 5550

Commit message: small updates
Connections:
- net GND: now also P5.1 (Pin_1)
Changed lines of the file:
@@
 Text Notes 600  7700 0    50   ~ 0
 AC608_HDMI_V2
+Wire Wire Line
+	5400 4800 5150 4800
 Wire Bus Line
 	6800 3400 6800 5550

Commit message: updated stamp
Connections:
- net GND: now also P4.1 (Pin_1)
- net R9: now also P3.4 (Pin_4); no longer P3.3 (Pin_3)
- net T8: now also P3.3 (Pin_3); no longer P3.2 (Pin_2)
- net T9: no longer P3.4 (Pin_4)
- new net R8: P3.2 (Pin_2)
Changed lines of the file:
@@
 	3400 4900 3650 4900
 Text Label 3550 5100 0    50   ~ 0
-T9
+R9
 Text Label 3550 5000 0    50   ~ 0
-R9
+T8
 Text Label 3550 4900 0    50   ~ 0
-T8
-Text Label 3550 4800 0    50   ~ 0
 R8
 $Sheet
@@
 F80 "P9" B R 2700 4900 50
 F81 "M10" B R 2700 4800 50
-F82 "LVDS_TX1_N" B R 2700 4700 50
-F83 "LVDS_TX1_P" B R 2700 4600 50
-F84 "LVDS_TX2_N" B R 2700 4500 50
-F85 "LVDS_TX2_P" B R 2700 4400 50
-F86 "LVDS_TX3_N" B R 2700 4300 50
-F87 "LVDS_TX3_P" B R 2700 4200 50
-F88 "LVDS_RXCLK_N" B R 2700 4100 50
-F89 "LVDS_RXCLK_P" B R 2700 4000 50
-F90 "LVDS_TX4_N" B R 2700 3900 50
-F91 "LVDS_TX4_P" B R 2700 3800 50
-F92 "LVDS_TX5_N" B R 2700 3700 50
-F93 "LVDS_TX5_P" B R 2700 3600 50
+F82 "J1" B R 2700 4700 50
+F83 "J2" B R 2700 4600 50
+F84 "K1" B R 2700 4500 50
+F85 "K2" B R 2700 4400 50
+F86 "L1" B R 2700 4300 50
+F87 "L2" B R 2700 4200 50
+F88 "M1" B R 2700 4100 50
+F89 "M2" B R 2700 4000 50
+F90 "N1" B R 2700 3900 50
+F91 "N2" B R 2700 3800 50
+F92 "P1" B R 2700 3700 50
+F93 "P2" B R 2700 3600 50
 F94 "R1" B R 2700 3500 50
 F95 "T2" B R 2700 3400 50
@@
 Wire Bus Line
 	3100 700  3100 6300
+$Comp
+L power:GND #PWR?
+U 1 1 5F9FCADC
+P 4950 4250
+F 0 "#PWR?" H 4950 4000 50  0001 C CNN
+F 1 "GND" V 4955 4122 50  0000 R CNN
+F 2 "" H 4950 4250 50  0001 C CNN
+F 3 "" H 4950 4250 50  0001 C CNN
+	1    4950 4250
+	0    1    1    0
+$EndComp
 $EndSCHEMATC
