File: hdmi.sch (KiCad schematic (older format))
At the start: 1 part

Commit message: first commit
Parts:
- removed U?: W25Q32JVSS, Package_SO:SOIC-8_5.23x5.23mm_P1.27mm, symbol Memory_Flash:W25Q32JVSS
- added C1, C2, C3, C4, C5, C6, C7, C8: C, symbol pspice:C
- added J1: HDMI_A_1.4, symbol Connector:HDMI_A_1.4
- added J? (x2): Conn_01x03, symbol Connector_Generic:Conn_01x03
Connections:
- net GND: now also J1.11 (CKS), J1.17 (GND), J1.2 (D2S), J1.5 (D1S), J1.8 (D0S), J1.SH
- new net: C1.1, J1.1 (D2+)
- new net: C7.1, J1.10 (CK+)
- new net: C8.1, J1.12 (CK-)
- new net: C2.1, J1.3 (D2-)
- new net: C3.1, J1.4 (D1+)
- new net: C4.1, J1.6 (D1-)
- new net: C5.1, J1.7 (D0+)
- new net: C6.1, J1.9 (D0-)
- new net ch0_n: C6.2
- new net ch0_p: C5.2
- new net ch1_n: C4.2
- new net ch1_p: C3.2
- new net ch2_n: C2.2
- new net ch2_p: C1.2
- new net clk_n: C8.2
- new net clk_p: C7.2

Commit message: first commit
Parts:
- added R4, R5, R6: 10k, symbol Device:R
- gave numbers to parts that had none: 2
Connections:
- net GND: now also J2.2 (Pin_2), R6.1
- net at J1.15 (SCL): now also R4.1
- net at J1.16 (SDA): now also R5.2
- net +5V: now reaches J1.18 (+5V)
- net +5V: now also J1.2 (Pin_2), R4.2, R5.1
- net at J1.19 (HPD/HEAC-): now also R6.2
- net RCKP: now reaches J1.1 (Pin_1)
- net TX1N: now reaches J1.3 (Pin_3)
- net RCKN: now reaches J2.1 (Pin_1)
- net TX1P: now reaches J2.3 (Pin_3)
- net ch0_n renamed TD0N
- net ch0_p renamed TD0P
- net ch1_n renamed TD1N
- net ch1_p renamed TD1P
- net ch2_n renamed TD2N
- net ch2_p renamed TD2P
- net clk_n renamed TCKN
- net clk_p renamed TCKP
Other:
- moved on the sheet: C1, C2, C3, C4, C5, C6, C7, C8, J1, J2
