File: camera.sch (KiCad schematic (older format))
At the start: 4 parts, among them P8 CAMERA

Commit message: peripheries updated
Other:
- moved on the sheet: R7

Commit message: small updates
Parts:
- C9: value C -> 0.1uF
Changed lines of the file:
@@
 P 4650 2950
 F 0 "C9" H 4535 2904 50  0000 R CNN
-F 1 "C" H 4535 2995 50  0000 R CNN
+F 1 "0.1uF" H 4535 2995 50  0000 R CNN
 F 2 "" H 4688 2800 50  0001 C CNN
 F 3 "~" H 4650 2950 50  0001 C CNN
