File: stamp_hole.sch (KiCad schematic (older format))
At the start: 1 part

Commit message: peripheries updated
Parts:
- added U?: W9825G6EH-6, WIN_TSOP-54_WIN, symbol 2020-10-25_15-23-21:W9825G6EH-6
- added U?: W25Q16JVSNIQ, SOIC_150MIL_WIN, symbol 2020-10-25_15-19-51:W25Q16JVSNIQ
Other:
- note added: "AC608 v1.3"
Changed lines of the file:
@@
 encoding utf-8
 Sheet 2 4
-Title ""
-Date ""
-Rev ""
-Comp ""
-Comment1 ""
+Title "AC608 development kit"
+Date "2020-10-25"
+Rev "v1.0"
+Comp "Pavol Risa"
+Comment1 "https://github.com/risapav/ac608"
 Comment2 ""
 Comment3 ""
@@
 $EndDescr
 $Bitmap
-Pos 10000 5350
+Pos 10200 1650
 Scale 1.000000
 Data
@@
 	1    0    0    -1
 $EndComp
+Text Notes 700  7650 0    50   ~ 0
+AC608 v1.3
+$Comp
+L 2020-10-25_15-23-21:W9825G6EH-6 U?
+U 1 1 5F9E6213
+P 8100 3400
+F 0 "U?" H 9400 3787 60  0000 C CNN
+F 1 "W9825G6EH-6" H 9400 3681 60  0000 C CNN
+F 2 "WIN_TSOP-54_WIN" H 9400 3640 60  0001 C CNN
+F 3 "" H 8100 3400 60  0000 C CNN
+	1    8100 3400
+	1    0    0    -1
+$EndComp
+$Comp
+L 2020-10-25_15-19-51:W25Q16JVSNIQ U?
+U 1 1 5F9E8255
+P 7250 850
+F 0 "U?" H 8850 1337 60  0000 C CNN
+F 1 "W25Q16JVSNIQ" H 8850 1231 60  0000 C CNN
+F 2 "SOIC_150MIL_WIN" H 8850 1190 60  0001 C CNN
+F 3 "" H 7250 850 60  0000 C CNN
+	1    7250 850
+	1    0    0    -1
+$EndComp

Commit message: updated stamp
Changed lines of the file:
@@
 M10
 Text HLabel 1000 2800 0    50   BiDi ~ 0
-LVDS_TX1_N
+J1
 Text HLabel 1500 2820 0    50   BiDi ~ 0
-LVDS_TX1_P
+J2
 Text HLabel 2000 2840 0    50   BiDi ~ 0
-LVDS_TX2_N
+K1
 Text HLabel 2550 2860 0    50   BiDi ~ 0
-LVDS_TX2_P
+K2
 Text HLabel 1000 2880 0    50   BiDi ~ 0
-LVDS_TX3_N
+L1
 Text HLabel 1500 2900 0    50   BiDi ~ 0
-LVDS_TX3_P
+L2
 Text HLabel 2000 2920 0    50   BiDi ~ 0
-LVDS_RXCLK_N
+M1
 Text HLabel 2550 2940 0    50   BiDi ~ 0
-LVDS_RXCLK_P
+M2
 Text HLabel 1000 2960 0    50   BiDi ~ 0
-LVDS_TX4_N
+N1
 Text HLabel 1500 2980 0    50   BiDi ~ 0
-LVDS_TX4_P
+N2
 Text HLabel 2000 3000 0    50   BiDi ~ 0
-LVDS_TX5_N
+P1
 Text HLabel 2550 3020 0    50   BiDi ~ 0
-LVDS_TX5_P
+P2
 Text HLabel 1000 3040 0    50   BiDi ~ 0
 R1
